Commit message: movement optimization

File: src/robotanik_sim/urdf/robotanik.urdf (robot description, URDF)
Before this commit: robot robotanik, 10 links, 9 joints
Links:
- removed link caster_wheel
- removed link left_wheel
- removed link right_wheel
- removed link sonar_link
- added link front_left_caster, mass 0.3; collision cylinder length=0.058 radius=0.065; visual cylinder length=0.058 radius=0.065
- added link front_right_caster, mass 0.3; collision cylinder length=0.058 radius=0.065; visual cylinder length=0.058 radius=0.065
- added link rear_left_wheel, mass 0.5; collision cylinder length=0.058 radius=0.065; visual cylinder length=0.058 radius=0.065
- added link rear_right_wheel, mass 0.5; collision cylinder length=0.058 radius=0.065; visual cylinder length=0.058 radius=0.065
- link base_link: mass 5.0 -> 15.0; geometry collision box size=0.50 0.35 0.30; visual box size=0.50 0.35 0.30
Joints:
- removed joint caster_joint
- removed joint left_wheel_joint
- removed joint right_wheel_joint
- removed joint sonar_joint
- added joint front_left_caster_joint: type fixed, parent base_link, child front_left_caster, origin xyz=0.15 0.204 -0.15 rpy=-1.5708 0 0
- added joint front_right_caster_joint: type fixed, parent base_link, child front_right_caster, origin xyz=0.15 -0.204 -0.15 rpy=1.5708 0 0
- added joint rear_left_wheel_joint: type continuous, parent base_link, child rear_left_wheel, origin xyz=-0.15 0.204 -0.15 rpy=-1.5708 0 0, axis 0 0 1
- added joint rear_right_wheel_joint: type continuous, parent base_link, child rear_right_wheel, origin xyz=-0.15 -0.204 -0.15 rpy=1.5708 0 0, axis 0 0 -1
- joint base_footprint_joint: origin xyz=0 0 0 rpy=0 0 0 -> xyz=0 0 0.215 rpy=0 0 0
- joint sonar_back_joint: origin xyz=-0.2 0 0 rpy=0 0 3.14159 -> xyz=-0.26 0 0.05 rpy=0 0 3.14159
- joint sonar_front_center_joint: origin xyz=0.2 0 0 rpy=0 0 0 -> xyz=0.26 0 0.05 rpy=0 0 0
- joint sonar_front_left_joint: origin xyz=0.2 0.15 0 rpy=0 0 0.52 -> xyz=0.20 0.175 0.05 rpy=0 0 0.785
- joint sonar_front_right_joint: origin xyz=0.2 -0.15 0 rpy=0 0 -0.52 -> xyz=0.20 -0.175 0.05 rpy=0 0 -0.785

Commit message: autonomous driving optimization

File: src/robotanik_sim/urdf/robotanik.urdf (robot description, URDF)
Before this commit: robot robotanik, 10 links, 9 joints
Links:
- removed link front_left_caster
- removed link front_right_caster
- removed link rear_left_wheel
- removed link rear_right_wheel
- added link left_caster_wheel, mass 0.2; collision sphere radius=0.0275; visual sphere radius=0.0275
- added link left_wheel, mass 0.5; collision cylinder length=0.058 radius=0.065; visual cylinder length=0.058 radius=0.065
- added link right_caster_wheel, mass 0.2; collision sphere radius=0.0275; visual sphere radius=0.0275
- added link right_wheel, mass 0.5; collision cylinder length=0.058 radius=0.065; visual cylinder length=0.058 radius=0.065
- link base_link: geometry collision box size=0.40 0.30 0.325; visual box size=0.40 0.30 0.325
Joints:
- removed joint front_left_caster_joint
- removed joint front_right_caster_joint
- removed joint rear_left_wheel_joint
- removed joint rear_right_wheel_joint
- added joint left_caster_joint: type fixed, parent base_link, child left_caster_wheel, origin xyz=0.15 0.10 -0.19 rpy=0 0 0
- added joint left_wheel_joint: type continuous, parent base_link, child left_wheel, origin xyz=-0.135 0.121 -0.1525 rpy=-1.5708 0 0, axis 0 0 1
- added joint right_caster_joint: type fixed, parent base_link, child right_caster_wheel, origin xyz=0.15 -0.10 -0.19 rpy=0 0 0
- added joint right_wheel_joint: type continuous, parent base_link, child right_wheel, origin xyz=-0.135 -0.121 -0.1525 rpy=1.5708 0 0, axis 0 0 -1
- joint sonar_back_joint: origin xyz=-0.26 0 0.05 rpy=0 0 3.14159 -> xyz=-0.21 0 0.05 rpy=0 0 3.14159
- joint sonar_front_center_joint: origin xyz=0.26 0 0.05 rpy=0 0 0 -> xyz=0.21 0 0.05 rpy=0 0 0
- joint sonar_front_left_joint: origin xyz=0.20 0.175 0.05 rpy=0 0 0.785 -> xyz=0.21 0.125 0.05 rpy=0 0 0.698
- joint sonar_front_right_joint: origin xyz=0.20 -0.175 0.05 rpy=0 0 -0.785 -> xyz=0.21 -0.125 0.05 rpy=0 0 -0.698
